File: training_board/training_board.kicad_sch (KiCad schematic)
At the start: 0 parts

Commit message: Pretty Cool Schematic
Hi Will
Parts:
- added D1, D2: GREEN, symbol Device:LED
- added J1: Molex_Megafit_02, MRDT_Connectors:MOLEX_MegaFit_02_Horizontal, symbol MRDT_Connectors:Molex_Megafit_02
- added R1: 330, symbol Device:R_US
- added R2: 6k8, symbol Device:R_US
- added U2: (no value), MRDT_Shields:RoveNode_H5, symbol MRDT_Shields:RoveNode_H5
Connections:
- new net: D1.2 (A), R1.2
- new net: D2.2 (A), R2.2
- new net +24V: J1.1, R2.1
- new net +3V3: R1.1
- new net GND: D1.1 (K), D2.1 (K), J1.2
Other:
- added sheet Power (Power.kicad_sch)

Commit message: Cleaned up a bit
Parts:
- added C5: C, symbol Device:C
- added C6: 0.1uF, symbol Device:C
- added H1, H2, H3, H4: MountingHole_Pad, Module:Maple_Mini, symbol Mechanical:MountingHole_Pad
- added J2: Conn_01x02_Pin, symbol Connector:Conn_01x02_Pin
- added J3: RJ45_LED_Shielded, Connector_RJ:RJ45_Abracon_ARJP11A-MA_Horizontal, symbol Connector:RJ45_LED_Shielded
- added R3: R_US, Resistor_THT:R_Array_SIP4, symbol Device:R_US
- added U3: SN65HVD232, Package_SO:SOIC-8_3.9x4.9mm_P1.27mm, symbol Interface_CAN_LIN:SN65HVD232
Connections:
- net +24V: now also U2.1 (VIN)
- net +3V3: now also C5.1, U3.3 (VCC)
- net GND: now also C5.2, C6.2, H1.1, H2.1, H3.1, H4.1, J3.11, J3.8, J3.9, J3.SH, U3.2 (GND)
- net CAN_TX: now reaches U2.12 (PA8)
- net CAN_TX: now also U3.1 (D)
- net CAN_RX: now reaches U2.13 (PC9)
- net CAN_RX: now also U3.4 (R)
- net RX+: now reaches U2.19 (RX+)
- net RX+: now also J3.4
- net RX-: now reaches U2.20 (RX-)
- net RX-: now also J3.6
- net TX+: now reaches U2.21 (TX+)
- net TX+: now also J3.1
- net TX-: now reaches U2.22 (TX-)
- net TX-: now also J3.3
- net LED2: now reaches U2.23 (LED2)
- net LED2: now also J3.10
- net LED1: now reaches U2.24 (LED1)
- net LED1: now also J3.12
- new net: C6.1, J3.2, J3.5
- new net: J2.1 (Pin_1), R3.2, U3.6 (CANL)
- new net: J2.2 (Pin_2), R3.1, U3.7 (CANH)
- no-connect marks 0 -> 37
Other:
- moved on the sheet: U2
