File: training_board/training_board.kicad_sch (KiCad schematic)
At the start: 0 parts

Commit message: Finished Schematic
A beautiful schematic
works
🙂🙂🙂🙂
Parts:
- added C1, C2: 0.1uF, Package_TO_SOT_SMD:TSOT-23-6, symbol Device:C
- added D1, D2: GRN, symbol Device:LED
- added H1, H2, H3, H4: MountingHole_Pad, MRDT_Drill_Holes:4_40_Hole_Pad_Via, symbol Mechanical:MountingHole_Pad
- added J1: Molex_Megafit_02, MRDT_Connectors:MOLEX_MegaFit_02_Horizontal, symbol MRDT_Connectors:Molex_Megafit_02
- added J2: Conn_01x02_Pin, symbol Connector:Conn_01x02_Pin
- added J3: RJ45_LED_Shielded, Connector_RJ:RJ45_Abracon_ARJP11A-MA_Horizontal, symbol Connector:RJ45_LED_Shielded
- added R1: 330, Resistor_THT:R_Array_SIP4, symbol Device:R_US
- added R2: 6k8, Resistor_THT:R_Array_SIP4, symbol Device:R_US
- added R3: 120, Resistor_THT:R_Array_SIP4, symbol Device:R_US
- added U1: (no value), MRDT_Shields:RoveNode_H5, symbol MRDT_Shields:RoveNode_H5
- added U3: SN65HVD232, Package_SO:SOIC-8_3.9x4.9mm_P1.27mm, symbol Interface_CAN_LIN:SN65HVD232
Connections:
- new net: C2.1, J3.2, J3.5
- new net: D2.1 (K), R2.1
- new net: J2.2 (Pin_2), R3.1, U3.7 (CANH)
- new net: J2.1 (Pin_1), R3.2, U3.6 (CANL)
- new net: D1.1 (K), R1.1
- new net +24V: D2.2 (A), J1.2, U1.1 (VIN)
- new net +3V3: C1.1, D1.2 (A), U1.3 (3V3), U3.3 (VCC)
- new net CAN_RX: U1.13 (PC9)
- new net CAN_TX: U1.12 (PA8), U3.1 (D)
- new net GND: C1.2, C2.2, H1.1, H2.1, H3.1, H4.1, J1.1, J3.11, J3.8, J3.9, J3.SH, R1.2, R2.2, U1.2 (GND), U3.2 (GND)
- new net LED1: J3.12, U1.24 (LED1)
- new net LED2: J3.10, U1.23 (LED2)
- new net RX+: J3.4, U1.19 (RX+)
- new net RX-: J3.6, U1.20 (RX-)
- new net TX+: J3.1, U1.21 (TX+)
- new net TX-: J3.3, U1.22 (TX-)
- no-connect marks 0 -> 1
Other:
- added sheet Power (Power.kicad_sch)

Commit message: PCB training
Parts:
- C1, C2: footprint Package_TO_SOT_SMD:TSOT-23-6 -> Capacitor_SMD:C_0603_1608Metric_Pad1.08x0.95mm_HandSolder
- D1, D2: footprint (none) -> Diode_SMD:D_0603_1608Metric_Pad1.05x0.95mm_HandSolder
- J2: footprint (none) -> Connector_JST:JST_PHD_B10B-PHDSS_2x05_P2.00mm_Vertical
- J3: footprint Connector_RJ:RJ45_Abracon_ARJP11A-MA_Horizontal -> MRDT_Connectors:RJ45_Teensy
- R1, R2, R3: footprint Resistor_THT:R_Array_SIP4 -> Resistor_SMD:R_0603_1608Metric_Pad0.98x0.95mm_HandSolder
Connections:
- net CAN_RX: now also U3.4 (R)
- no-connect marks 1 -> 35
Changed lines of the file:
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@@
 	)
 	(junction
-		(at 95.25 119.38)
-		(diameter 0)
-		(color 0 0 0 0)
-	)
-	(junction
 		(at 149.86 121.92)
 		(diameter 0)
@@
 	)
 	(no_connect
+		(at 160.02 55.88)
+	)
+	(no_connect
+		(at 160.02 77.47)
+	)
+	(no_connect
+		(at 184.15 46.99)
+	)
+	(no_connect
+		(at 184.15 43.18)
+	)
+	(no_connect
+		(at 184.15 77.47)
+	)
+	(no_connect
 		(at 251.46 138.43)
 	)
+	(no_connect
+		(at 184.15 49.53)
+	)
+	(no_connect
+		(at 184.15 59.69)
+	)
+	(no_connect
+		(at 160.02 85.09)
+	)
+	(no_connect
+		(at 160.02 36.83)
+	)
+	(no_connect
+		(at 160.02 46.99)
+	)
+	(no_connect
+		(at 160.02 44.45)
+	)
+	(no_connect
+		(at 160.02 69.85)
+	)
+	(no_connect
+		(at 184.15 54.61)
+	)
+	(no_connect
+		(at 184.15 72.39)
+	)
+	(no_connect
+		(at 184.15 52.07)
+	)
+	(no_connect
+		(at 160.02 82.55)
+	)
+	(no_connect
+		(at 160.02 58.42)
+	)
+	(no_connect
+		(at 160.02 52.07)
+	)
+	(no_connect
+		(at 160.02 62.23)
+	)
+	(no_connect
+		(at 160.02 39.37)
+	)
+	(no_connect
+		(at 160.02 67.31)
+	)
+	(no_connect
+		(at 184.15 74.93)
+	)
+	(no_connect
+		(at 184.15 57.15)
+	)
+	(no_connect
+		(at 184.15 67.31)
+	)
+	(no_connect
+		(at 160.02 72.39)
+	)
+	(no_connect
+		(at 160.02 34.29)
+	)
+	(no_connect
+		(at 160.02 49.53)
+	)
+	(no_connect
+		(at 160.02 64.77)
+	)
+	(no_connect
+		(at 160.02 41.91)
+	)
+	(no_connect
+		(at 184.15 69.85)
+	)
+	(no_connect
+		(at 160.02 31.75)
+	)
+	(no_connect
+		(at 184.15 40.64)
+	)
+	(no_connect
+		(at 160.02 80.01)
+	)
+	(no_connect
+		(at 160.02 74.93)
+	)
 	(wire
 		(pts
@@
 	(wire
 		(pts
+			(xy 109.22 124.46) (xy 115.57 124.46)
+		)
+		(stroke
+			(width 0)
+			(type default)
+		)
+	)
+	(wire
+		(pts
 			(xy 238.76 118.11) (xy 238.76 111.76)
 		)
@@
 	(wire
 		(pts
-			(xy 95.25 120.65) (xy 95.25 119.38)
-		)
-		(stroke
-			(width 0)
-			(type default)
-		)
-	)
-	(wire
-		(pts
 			(xy 193.04 34.29) (xy 184.15 34.29)
 		)
@@
 			)
 		)
-		(property "Footprint" "Package_TO_SOT_SMD:TSOT-23-6"
+		(property "Footprint" "Capacitor_SMD:C_0603_1608Metric_Pad1.08x0.95mm_HandSolder"
 			(at 239.7252 149.86 0)
 			(hide yes)
@@
 			)
 		)
-		(property "Footprint" "Resistor_THT:R_Array_SIP4"
+		(property "Footprint" "Resistor_SMD:R_0603_1608Metric_Pad0.98x0.95mm_HandSolder"
 			(at 243.586 52.324 90)
 			(hide yes)
@@
 			)
 		)
-		(property "Footprint" "Resistor_THT:R_Array_SIP4"
+		(property "Footprint" "Resistor_SMD:R_0603_1608Metric_Pad0.98x0.95mm_HandSolder"
 			(at 150.876 125.984 90)
 			(hide yes)
@@
 			)
 		)
-		(property "Footprint" ""
+		(property "Footprint" "Diode_SMD:D_0603_1608Metric_Pad1.05x0.95mm_HandSolder"
 			(at 242.57 41.91 0)
 			(hide yes)
@@
 			)
 		)
-		(property "Footprint" ""
+		(property "Footprint" "Diode_SMD:D_0603_1608Metric_Pad1.05x0.95mm_HandSolder"
 			(at 218.44 41.91 0)
 			(hide yes)
@@
 			)
 		)
-		(property "Footprint" "Connector_RJ:RJ45_Abracon_ARJP11A-MA_Horizontal"
+		(property "Footprint" "MRDT_Connectors:RJ45_Teensy"
 			(at 244.475 128.27 90)
 			(hide yes)
@@
 			)
 		)
-		(property "Footprint" ""
+		(property "Footprint" "Connector_JST:JST_PHD_B10B-PHDSS_2x05_P2.00mm_Vertical"
 			(at 165.1 127 0)
 			(hide yes)
@@
 			)
 		)
-		(property "Footprint" "Resistor_THT:R_Array_SIP4"
+		(property "Footprint" "Resistor_SMD:R_0603_1608Metric_Pad0.98x0.95mm_HandSolder"
 			(at 219.456 52.324 90)
 			(hide yes)
@@
 			)
 		)
-		(property "Footprint" "Package_TO_SOT_SMD:TSOT-23-6"
+		(property "Footprint" "Capacitor_SMD:C_0603_1608Metric_Pad1.08x0.95mm_HandSolder"
 			(at 96.2152 127 0)
 			(hide yes)
