File: training_board/training_board.kicad_sch (KiCad schematic)
At the start: 0 parts

Commit message: Finished Schematic
a description
100000000% working very goocosdfaljkdsnf;sdkjfasd;kljfnasd;lkf
Parts:
- added C2, C6: 0.1uF, symbol Device:C
- added D1, D2: GREEN, symbol Device:LED
- added H1, H2, H3, H4: MountingHole_Pad, symbol Mechanical:MountingHole_Pad
- added J1: Molex_Megafit_02, MRDT_Connectors:MOLEX_MegaFit_02_Horizontal, symbol MRDT_Connectors:Molex_Megafit_02
- added J2: Conn_01x02_Pin, symbol Connector:Conn_01x02_Pin
- added J3: RJ45_LED_Shielded, symbol Connector:RJ45_LED_Shielded
- added R1: 330, symbol Device:R_US
- added R2: 6k8, symbol Device:R_US
- added R3: 120, symbol Device:R_US
- added U2: (no value), MRDT_Shields:RoveNode_H5, symbol MRDT_Shields:RoveNode_H5
- added U3: SN65HVD232, Package_SO:SOIC-8_3.9x4.9mm_P1.27mm, symbol Interface_CAN_LIN:SN65HVD232
Connections:
- new net: D2.1 (K), R2.1
- new net: D1.1 (K), R1.1
- new net: J2.2 (Pin_2), R3.1, U3.7 (CANH)
- new net: J2.1 (Pin_1), R3.2, U3.6 (CANL)
- new net: C6.1, J3.2, J3.5
- new net +24V: D2.2 (A), J1.2, U2.1 (VIN)
- new net +3V3: C2.1, D1.2 (A), U2.3 (3V3), U3.3 (VCC)
- new net CAN_RX: U2.12 (PA8), U3.4 (R)
- new net CAN_TX: U2.13 (PC9), U3.1 (D)
- new net GND: C2.2, C6.2, H1.1, H2.1, H3.1, H4.1, J1.1, J3.11, J3.8, J3.9, J3.SH, R1.2, R2.2, U2.2 (GND), U3.2 (GND)
- new net LED1: J3.12, U2.24 (LED1)
- new net LED2: J3.10, U2.23 (LED2)
- new net RX+: J3.4, U2.19 (RX+)
- new net RX-: J3.6, U2.20 (RX-)
- new net TX+: J3.1, U2.21 (TX+)
- new net TX-: J3.3, U2.22 (TX-)
- no-connect marks 0 -> 109
Other:
- added sheet Power (power.kicad_sch)

Commit message: Finished a beautiful schematic for ya
Parts:
- C2, C6: footprint (none) -> Capacitor_SMD:C_0603_1608Metric_Pad1.08x0.95mm_HandSolder
- D1, D2: footprint (none) -> Diode_SMD:D_0603_1608Metric
- H1, H2, H3, H4: footprint (none) -> MRDT_Drill_Holes:4_40_Hole_Pad_Via
- J2: footprint (none) -> Connector_JST:JST_PH_S2B-PH-SM4-TB_1x02-1MP_P2.00mm_Horizontal
- J3: footprint (none) -> MRDT_Connectors:RJ45_Teensy
- R1, R2, R3: footprint (none) -> Resistor_SMD:R_0603_1608Metric_Pad0.98x0.95mm_HandSolder
Connections:
- no-connect marks 109 -> 35
Other:
- moved on the sheet: U2
