File: training_board/untitled.kicad_sch (KiCad schematic)
At the start: 5 parts

Commit message: Finished Schematic
and it is awesome and totally finished
Parts:
- removed Conn1: Molex_SL_02, symbol MRDT_Connectors:Molex_SL_02
- removed D1: LED, symbol Device:LED
- removed D2: GREEN, symbol Device:LED
- removed R1, R2: 330, symbol Device:R_US
- added C1: 10uF, symbol Device:C
- added C2: 0.1uF, symbol Device:C
- added C7, C8: 22uF, symbol Device:C
- added L1: 3.9uH, symbol Device:L
- added U1: AP63203WU, Package_TO_SOT_SMD:TSOT-23-6, symbol Regulator_Switching:AP63203WU
Connections:
- net +24V: now also U1.2 (EN), U1.3 (IN)
- net +3V3: now also C7.1, C8.1, L1.2, U1.1 (FB)
- net GND: now also C1.2, C7.2, C8.2
- new net: C2.2, L1.1, U1.6 (BST)
Other:
- removed sheet Power

Commit message: Made a Giga cool Turtle Board (again)
Parts:
- C1, C2, C7, C8: footprint (none) -> Capacitor_SMD:C_0603_1608Metric_Pad1.08x0.95mm_HandSolder
- L1: footprint (none) -> Inductor_SMD:L_1008_2520Metric_Pad1.43x2.20mm_HandSolder
Changed lines of the file:
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@@
 			)
 		)
-		(property "Footprint" ""
+		(property "Footprint" "Inductor_SMD:L_1008_2520Metric_Pad1.43x2.20mm_HandSolder"
 			(at 168.91 91.44 0)
 			(hide yes)
@@
 		(instances
 			(project "training_board"
-				(path "/c8b65c5a-76a4-40b3-a332-766a1070b56a"
-					(reference "L1")
-					(unit 1)
-				)
 				(path "/c8b65c5a-76a4-40b3-a332-766a1070b56a/642b35e5-5dba-49d9-abbd-8da8f0279939"
 					(reference "L1")
@@
 			)
 		)
-		(property "Footprint" ""
+		(property "Footprint" "Capacitor_SMD:C_0603_1608Metric_Pad1.08x0.95mm_HandSolder"
 			(at 119.0752 102.87 0)
 			(hide yes)
@@
 		(instances
 			(project "training_board"
-				(path "/c8b65c5a-76a4-40b3-a332-766a1070b56a"
-					(reference "C1")
-					(unit 1)
-				)
 				(path "/c8b65c5a-76a4-40b3-a332-766a1070b56a/642b35e5-5dba-49d9-abbd-8da8f0279939"
 					(reference "C1")
@@
 		(instances
 			(project "training_board"
-				(path "/c8b65c5a-76a4-40b3-a332-766a1070b56a"
-					(reference "#PWR05")
-					(unit 1)
-				)
 				(path "/c8b65c5a-76a4-40b3-a332-766a1070b56a/642b35e5-5dba-49d9-abbd-8da8f0279939"
 					(reference "#PWR05")
@@
 		(instances
 			(project "training_board"
-				(path "/c8b65c5a-76a4-40b3-a332-766a1070b56a"
-					(reference "U1")
-					(unit 1)
-				)
 				(path "/c8b65c5a-76a4-40b3-a332-766a1070b56a/642b35e5-5dba-49d9-abbd-8da8f0279939"
 					(reference "U1")
@@
 			)
 		)
-		(property "Footprint" ""
+		(property "Footprint" "Capacitor_SMD:C_0603_1608Metric_Pad1.08x0.95mm_HandSolder"
 			(at 182.5752 107.95 0)
 			(hide yes)
@@
 		(instances
 			(project "training_board"
-				(path "/c8b65c5a-76a4-40b3-a332-766a1070b56a"
-					(reference "C8")
-					(unit 1)
-				)
 				(path "/c8b65c5a-76a4-40b3-a332-766a1070b56a/642b35e5-5dba-49d9-abbd-8da8f0279939"
 					(reference "C8")
@@
 		(instances
 			(project "training_board"
-				(path "/c8b65c5a-76a4-40b3-a332-766a1070b56a"
-					(reference "#PWR04")
-					(unit 1)
-				)
 				(path "/c8b65c5a-76a4-40b3-a332-766a1070b56a/642b35e5-5dba-49d9-abbd-8da8f0279939"
 					(reference "#PWR04")
@@
 		(instances
 			(project "training_board"
-				(path "/c8b65c5a-76a4-40b3-a332-766a1070b56a"
-					(reference "#PWR02")
-					(unit 1)
-				)
 				(path "/c8b65c5a-76a4-40b3-a332-766a1070b56a/642b35e5-5dba-49d9-abbd-8da8f0279939"
 					(reference "#PWR02")
@@
 			)
 		)
-		(property "Footprint" ""
+		(property "Footprint" "Capacitor_SMD:C_0603_1608Metric_Pad1.08x0.95mm_HandSolder"
 			(at 157.1752 91.44 0)
 			(hide yes)
@@
 		(instances
 			(project "training_board"
-				(path "/c8b65c5a-76a4-40b3-a332-766a1070b56a"
-					(reference "C2")
-					(unit 1)
-				)
 				(path "/c8b65c5a-76a4-40b3-a332-766a1070b56a/642b35e5-5dba-49d9-abbd-8da8f0279939"
 					(reference "C2")
@@
 			)
 		)
-		(property "Footprint" ""
+		(property "Footprint" "Capacitor_SMD:C_0603_1608Metric_Pad1.08x0.95mm_HandSolder"
 			(at 157.1752 107.95 0)
 			(hide yes)
@@
 		(instances
 			(project "training_board"
-				(path "/c8b65c5a-76a4-40b3-a332-766a1070b56a"
-					(reference "C7")
-					(unit 1)
-				)
 				(path "/c8b65c5a-76a4-40b3-a332-766a1070b56a/642b35e5-5dba-49d9-abbd-8da8f0279939"
 					(reference "C7")
@@
 		(instances
 			(project "training_board"
-				(path "/c8b65c5a-76a4-40b3-a332-766a1070b56a"
+				(path "/c8b65c5a-76a4-40b3-a332-766a1070b56a/642b35e5-5dba-49d9-abbd-8da8f0279939"
 					(reference "#PWR03")
-					(unit 1)
-				)
-				(path "/c8b65c5a-76a4-40b3-a332-766a1070b56a/642b35e5-5dba-49d9-abbd-8da8f0279939"
-					(reference "#PWR03")
