File: training_board/power.kicad_sch (KiCad schematic)
At the start: 6 parts, among them U1 AP63203WU

Commit message: Finished a beautiful schematic for ya
Parts:
- C1, C3, C4, C5: footprint (none) -> Capacitor_SMD:C_0603_1608Metric_Pad1.08x0.95mm_HandSolder
- L1: footprint (none) -> Inductor_SMD:L_1008_2520Metric_Pad1.43x2.20mm_HandSolder
Changed lines of the file:
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@@
 		(instances
 			(project "training_board"
-				(path "/c8b65c5a-76a4-40b3-a332-766a1070b56a"
-					(reference "#PWR03")
-					(unit 1)
-				)
 				(path "/c8b65c5a-76a4-40b3-a332-766a1070b56a/140e784b-4a0e-46f9-9dee-6c27639aeef8"
 					(reference "#PWR03")
@@
 			)
 		)
-		(property "Footprint" ""
+		(property "Footprint" "Capacitor_SMD:C_0603_1608Metric_Pad1.08x0.95mm_HandSolder"
 			(at 136.8552 82.55 0)
 			(hide yes)
@@
 		(instances
 			(project "training_board"
-				(path "/c8b65c5a-76a4-40b3-a332-766a1070b56a"
-					(reference "#PWR05")
-					(unit 1)
-				)
 				(path "/c8b65c5a-76a4-40b3-a332-766a1070b56a/140e784b-4a0e-46f9-9dee-6c27639aeef8"
 					(reference "#PWR05")
@@
 		(instances
 			(project "training_board"
-				(path "/c8b65c5a-76a4-40b3-a332-766a1070b56a"
-					(reference "U1")
-					(unit 1)
-				)
 				(path "/c8b65c5a-76a4-40b3-a332-766a1070b56a/140e784b-4a0e-46f9-9dee-6c27639aeef8"
 					(reference "U1")
@@
 			)
 		)
-		(property "Footprint" ""
+		(property "Footprint" "Capacitor_SMD:C_0603_1608Metric_Pad1.08x0.95mm_HandSolder"
 			(at 169.8752 97.79 0)
 			(hide yes)
@@
 		(instances
 			(project "training_board"
-				(path "/c8b65c5a-76a4-40b3-a332-766a1070b56a"
-					(reference "#PWR06")
-					(unit 1)
-				)
 				(path "/c8b65c5a-76a4-40b3-a332-766a1070b56a/140e784b-4a0e-46f9-9dee-6c27639aeef8"
 					(reference "#PWR06")
@@
 		(instances
 			(project "training_board"
-				(path "/c8b65c5a-76a4-40b3-a332-766a1070b56a"
-					(reference "#PWR07")
-					(unit 1)
-				)
 				(path "/c8b65c5a-76a4-40b3-a332-766a1070b56a/140e784b-4a0e-46f9-9dee-6c27639aeef8"
 					(reference "#PWR07")
@@
 			)
 		)
-		(property "Footprint" ""
+		(property "Footprint" "Capacitor_SMD:C_0603_1608Metric_Pad1.08x0.95mm_HandSolder"
 			(at 91.1352 93.98 0)
 			(hide yes)
@@
 		(instances
 			(project "training_board"
-				(path "/c8b65c5a-76a4-40b3-a332-766a1070b56a"
-					(reference "C1")
-					(unit 1)
-				)
 				(path "/c8b65c5a-76a4-40b3-a332-766a1070b56a/140e784b-4a0e-46f9-9dee-6c27639aeef8"
 					(reference "C1")
@@
 		(instances
 			(project "training_board"
-				(path "/c8b65c5a-76a4-40b3-a332-766a1070b56a"
-					(reference "#PWR04")
-					(unit 1)
-				)
 				(path "/c8b65c5a-76a4-40b3-a332-766a1070b56a/140e784b-4a0e-46f9-9dee-6c27639aeef8"
 					(reference "#PWR04")
@@
 			)
 		)
-		(property "Footprint" ""
+		(property "Footprint" "Capacitor_SMD:C_0603_1608Metric_Pad1.08x0.95mm_HandSolder"
 			(at 157.1752 97.79 0)
 			(hide yes)
@@
 			)
 		)
-		(property "Footprint" ""
+		(property "Footprint" "Inductor_SMD:L_1008_2520Metric_Pad1.43x2.20mm_HandSolder"
 			(at 149.86 85.09 0)
 			(hide yes)
@@
 		(instances
 			(project "training_board"
-				(path "/c8b65c5a-76a4-40b3-a332-766a1070b56a"
+				(path "/c8b65c5a-76a4-40b3-a332-766a1070b56a/140e784b-4a0e-46f9-9dee-6c27639aeef8"
 					(reference "L1")
-					(unit 1)
-				)
-				(path "/c8b65c5a-76a4-40b3-a332-766a1070b56a/140e784b-4a0e-46f9-9dee-6c27639aeef8"
-					(reference "L1")
